Commit message: add: e1 sim2sim scripts and interrupt env

File: data/robots/droidrobot/E1/E1_21dof.urdf (robot description, URDF)
Before this commit: robot E1_v2, 20 links, 19 joints
Links:
- added link left_elbow_link, mass 0.5; collision mesh filename=meshes/left_elbow_link.STL; visual mesh filename=meshes/left_elbow_link.STL
- added link right_elbow_link, mass 0.5; collision mesh filename=meshes/right_elbow_link.STL; visual mesh filename=meshes/right_elbow_link.STL
Joints:
- added joint left_elbow_joint: type revolute, parent left_shoulder_yaw_link, child left_elbow_link, origin xyz=0 0 -0.153 rpy=0 0 0, axis 0 1 0, limit lower=-0.6981 upper=1.5708 effort=36 velocity=50.27
- added joint right_elbow_joint: type revolute, parent right_shoulder_yaw_link, child right_elbow_link, origin xyz=0 0 -0.153 rpy=0 0 0, axis 0 1 0, limit lower=-0.6981 upper=1.5708 effort=36 velocity=50.27
- joint left_shoulder_pitch_joint: type fixed -> revolute
- joint left_shoulder_roll_joint: type fixed -> revolute
- joint left_shoulder_yaw_joint: type fixed -> revolute
- joint right_shoulder_pitch_joint: type fixed -> revolute
- joint right_shoulder_roll_joint: type fixed -> revolute
- joint right_shoulder_yaw_joint: type fixed -> revolute
- joint waist_yaw_joint: type fixed -> revolute
